File: low volt board - NL  S-3C-v2.kicad_sch (KiCad schematic)
At the start: 42 parts, among them J1 ESP32-S3-ETH-WAVETREE-Footpri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, J2 ILI9341 TFT 2.8" Display with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, J3 4 Channel 5v Relay Connector, J4 SPDT (on)-off-(on), J5 ADC Inputs - 24v side, J6 Dry Contact OptoCoupler, J8 5vIn, Q1-Buzzer1 S8050, SW1 SW_SPDT, U1 ADS1115IDGS - low volt, U2 ADS1115IDGS - 24v, U3-Opto1 PC817

Commit message: Final design before first autoroute
Co-Authored-By: Claude Opus 4.6 <noreply@anthropic.com>
Connections:
- net +5V: now also J3.6 (5v), J8.2 (Pin_2); no longer J3.1 (5v), J8.1 (Pin_1)
- net A1-2-E: no longer J5.6 (A1-3)
- net A1-3-E: now also J5.6 (A1-3)
- net A2-1: now also R8-A2-1.2; no longer R8-A2-1.1
- net A2-1-E: now also R8-A2-1.1; no longer R8-A2-1.2
- net A2-2: now also R9-A2-2.2; no longer R9-A2-2.1
- net A2-2-E: now also R9-A2-2.1; no longer R9-A2-2.2
- net GND: now also J3.5 (GND), J8.1 (Pin_1); no longer J3.2 (GND), J8.2 (Pin_2)
- net IO15: now also J3.2 (IN3); no longer J3.5 (IN3)
- net IO16: now also J3.4 (IN1); no longer J3.3 (IN1)
- net IO18: now also J3.3 (IN2); no longer J3.4 (IN2)
- net IO3: now also J3.1 (IN4); no longer J3.6 (IN4)
- net Buzzer-2: now reaches Q1-Buzzer1.2 (B), R1-Buzzer1.2
- net Buzzer-3: now reaches LS1-Buzzer1.3 (-LEAD), Q1-Buzzer1.3 (C)
- net IO21 renamed Buzer-IO21
Other:
- moved on the sheet: C1, C2, C3, C4, C5, R10-A2-3, R17-A1-3, R18-A1-2, R8-A2-1, R9-A2-2

Commit message: Traces and DRC passing - still need mounting holes
Co-Authored-By: Claude Opus 4.6 <noreply@anthropic.com>
Parts:
- LS1-Buzzer1: footprint MLT8530 -> MLT-8530:MLT8530
Changed lines of the file:
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@@
 			)
 		)
-		(property "Footprint" "MLT8530"
+		(property "Footprint" "MLT-8530:MLT8530"
 			(at 179.07 229.54 0)
 			(effects

Commit message: Traces and DRC passing - still need mounting holes
Co-Authored-By: Claude Opus 4.6 <noreply@anthropic.com>
Parts:
- added H1, H2: MountingHole, MountingHole:MountingHole_4.3mm_M4_DIN965_Pad, symbol Mechanical:MountingHole
Changed lines of the file:
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@@
+	)
+	(symbol
+		(lib_id "Mechanical:MountingHole")
+		(at 171.45 86.36 0)
+		(unit 1)
+		(exclude_from_sim no)
+		(in_bom no)
+		(on_board yes)
+		(dnp no)
+		(fields_autoplaced yes)
+		(property "Reference" "H1"
+			(at 173.99 85.0899 0)
+			(effects
+				(font
+					(size 1.27 1.27)
+				)
+				(justify left)
+			)
+		)
+		(property "Value" "MountingHole"
+			(at 173.99 87.6299 0)
+			(effects
+				(font
+					(size 1.27 1.27)
+				)
+				(justify left)
+			)
+		)
+		(property "Footprint" "MountingHole:MountingHole_4.3mm_M4_DIN965_Pad"
+			(at 171.45 86.36 0)
+			(effects
+				(font
+					(size 1.27 1.27)
+				)
+				(hide yes)
+			)
+		)
+		(property "Datasheet" "~"
+			(at 171.45 86.36 0)
+			(effects
+				(font
+					(size 1.27 1.27)
+				)
+				(hide yes)
+			)
+		)
+		(property "Description" "Mounting Hole without connection"
+			(at 171.45 86.36 0)
+			(effects
+				(font
+					(size 1.27 1.27)
+				)
+				(hide yes)
+			)
+		)
+		(instances
+			(project ""
+				(path "/9df24c09-b453-48f7-b96a-68d109fc3890"
+					(reference "H1")
+					(unit 1)
+				)
+			)
+		)
 	)
 	(symbol
@@
 					(unit 1)
 				)
+			)
+		)
+	)
+	(symbol
+		(lib_id "Mechanical:MountingHole")
+		(at 171.45 100.33 0)
+		(unit 1)
+		(exclude_from_sim no)
+		(in_bom no)
+		(on_board yes)
+		(dnp no)
+		(fields_autoplaced yes)
+		(property "Reference" "H2"
+			(at 173.99 99.0599 0)
+			(effects
+				(font
+					(size 1.27 1.27)
+				)
+				(justify left)
+			)
+		)
+		(property "Value" "MountingHole"
+			(at 173.99 101.5999 0)
+			(effects
+				(font
+					(size 1.27 1.27)
+				)
+				(justify left)
+			)
+		)
+		(property "Footprint" "MountingHole:MountingHole_4.3mm_M4_DIN965_Pad"
+			(at 171.45 100.33 0)
+			(effects
+				(font
+					(size 1.27 1.27)
+				)
+				(hide yes)
+			)
+		)
+		(property "Datasheet" "~"
+			(at 171.45 100.33 0)
+			(effects
+				(font
+					(size 1.27 1.27)
+				)
+				(hide yes)
+			)
+		)
+		(property "Description" "Mounting Hole without connection"
+			(at 171.45 100.33 0)
+			(effects
+				(font
+					(size 1.27 1.27)
+				)
+				(hide yes)
+			)
+		)
+		(instances
+			(project ""
+				(path "/9df24c09-b453-48f7-b96a-68d109fc3890"
+					(reference "H2")
+					(unit 1)
+				)

Commit message: Fixed footprint issues
Co-Authored-By: Claude Opus 4.6 <noreply@anthropic.com>
Parts:
- J2: footprint Connector_PinHeader_1.00mm:PinHeader_1x13_P1.00mm_Vertical -> Connector_PinHeader_2.54mm:PinHeader_1x13_P2.54mm_Vertical
- Q1-Buzzer1: footprint Package_TO_SOT_THT:TO-92_Inline -> Package_TO_SOT_SMD:SOT-23
Changed lines of the file:
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@@
 			)
 		)
-		(property "Footprint" "Package_TO_SOT_THT:TO-92_Inline"
+		(property "Footprint" "Package_TO_SOT_SMD:SOT-23"
 			(at 143.51 146.685 0)
 			(effects
@@
 			)
 		)
-		(property "Footprint" "Connector_PinHeader_1.00mm:PinHeader_1x13_P1.00mm_Vertical"
+		(property "Footprint" "Connector_PinHeader_2.54mm:PinHeader_1x13_P2.54mm_Vertical"
 			(at 140.97 45.72 0)
 			(effects

Commit message: Minor fixes including missing nets
Co-Authored-By: Claude Opus 4.6 <noreply@anthropic.com>
Connections:
- net 3v Clean is gone; now on net +3.3V: LS1-Buzzer1.2 (+LEAD)
- net GND - 3v Clean is gone; now on net GND: R2-Throw-A1.2, R3-ThrowB1.2
- net IO17 is gone; now on net A1-0: J4.2 (Common), R4-Common1.1
- net SCD is gone; now on net SDA: J1.21 (GPIO43_(UART0_TX))
- net +3.3V: now also J1.10 (GPIO41)
- net GND: now also J1.13 (GND), J1.30 (CHIP_UP), J1.33 (GND), J1.8 (GND)

Commit message: Ready for fabrication review
Co-Authored-By: Claude Opus 4.6 <noreply@anthropic.com>
Connections:
- net +3.3V: no longer J1.10 (GPIO41), R5.1, U1.2 (ALERT/RDY), U2.2 (ALERT/RDY)
- net GND: now also J1.28 (GND), Q1-Buzzer1.2 (B); no longer Q1-Buzzer1.1 (E)
- net SCL: no longer R6-SCL1.1, U1.10 (SCL), U2.10 (SCL)
- net SDA: no longer R7-SDA1.1, U1.9 (SDA), U2.9 (SDA)
- net Buzer-IO21: no longer names the net of R1-Buzzer1.1
- net Buzer-IO21: now also Q1-Buzzer1.1 (E); no longer J1.35 (GPIO21)
- net Buzzer-2 renamed IO21
- net IO21: now also J1.35 (GPIO21); no longer Q1-Buzzer1.2 (B)
- net Buzzer-3: no longer names the net of LS1-Buzzer1.3 (-LEAD), Q1-Buzzer1.3 (C)
- new net IO41: J1.10 (GPIO41), R5.1, U1.2 (ALERT/RDY), U2.2 (ALERT/RDY)
- new net SCL-In: R6-SCL1.1, U1.10 (SCL), U2.10 (SCL)
- new net SDA-In: R7-SDA1.1, U1.9 (SDA), U2.9 (SDA)
Other:
- moved on the sheet: Q1-Buzzer1, R1-Buzzer1

Commit message: v2 ready for production
Co-Authored-By: Claude Opus 4.6 <noreply@anthropic.com>
Connections:
- net +3.3V: now also R6-SCL1.1, R7-SDA1.1
- net SCL: now also U1.10 (SCL), U2.10 (SCL)
- net SDA: now also U1.9 (SDA), U2.9 (SDA)
- removed net SCL-In: R6-SCL1.1, U1.10 (SCL), U2.10 (SCL)
- removed net SDA-In: R7-SDA1.1, U1.9 (SDA), U2.9 (SDA)
Changed lines of the file:
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@@
 		)
 	)
-	(label "SCL-In"
-		(at 64.77 185.42 180)
-		(effects
-			(font
-				(size 1.27 1.27)
-			)
-			(justify right bottom)
-		)
-	)
 	(label "A2-0"
 		(at 92.71 172.72 180)
@@
 		)
 	)
-	(label "SCL-In"
+	(label "SCL"
 		(at 54.61 186.69 270)
 		(effects
@@
 		)
 	)
-	(label "SDA-In"
+	(label "SDA"
 		(at 50.8 186.69 270)
 		(effects
@@
 		)
 	)
-	(label "SCL-In"
+	(label "SCL"
 		(at 124.46 185.42 270)
 		(effects
@@
 		)
 	)
-	(label "SDA-In"
-		(at 64.77 194.31 180)
-		(effects
-			(font
-				(size 1.27 1.27)
-			)
-			(justify right bottom)
-		)
-	)
 	(label "IO21"
 		(at 157.48 147.32 0)
@@
 		)
 	)
-	(label "SDA-In"
+	(label "SDA"
 		(at 120.65 185.42 270)
 		(effects
@@
 	)
 	(symbol
+		(lib_id "power:+3.3V")
+		(at 64.77 185.42 90)
+		(unit 1)
+		(exclude_from_sim no)
+		(in_bom yes)
+		(on_board yes)
+		(dnp no)
+		(fields_autoplaced yes)
+		(property "Reference" "#PWR039"
+			(at 68.58 185.42 0)
+			(effects
+				(font
+					(size 1.27 1.27)
+				)
+				(hide yes)
+			)
+		)
+		(property "Value" "+3.3V"
+			(at 60.96 185.4199 90)
+			(effects
+				(font
+					(size 1.27 1.27)
+				)
+				(justify left)
+			)
+		)
+		(property "Footprint" ""
+			(at 64.77 185.42 0)
+			(effects
+				(font
+					(size 1.27 1.27)
+				)
+				(hide yes)
+			)
+		)
+		(property "Datasheet" ""
+			(at 64.77 185.42 0)
+			(effects
+				(font
+					(size 1.27 1.27)
+				)
+				(hide yes)
+			)
+		)
+		(property "Description" "Power symbol creates a global label with name \"+3.3V\""
+			(at 64.77 185.42 0)
+			(effects
+				(font
+					(size 1.27 1.27)
+				)
+				(hide yes)
+			)
+		)
+		(pin "1"
+		)
+		(instances
+			(project ""
+				(path "/9df24c09-b453-48f7-b96a-68d109fc3890"
+					(reference "#PWR039")
+					(unit 1)
+				)
+			)
+		)
+	)
+	(symbol
 		(lib_id "power:GND")
 		(at 104.3 74.93 90)
@@
 					(unit 1)
 				)
+			)
+		)
+	)
+	(symbol
+		(lib_id "power:+3.3V")
+		(at 64.77 194.31 90)
+		(unit 1)
+		(exclude_from_sim no)
+		(in_bom yes)
+		(on_board yes)
+		(dnp no)
+		(fields_autoplaced yes)
+		(property "Reference" "#PWR040"
+			(at 68.58 194.31 0)
+			(effects
+				(font
+					(size 1.27 1.27)
+				)
+				(hide yes)
+			)
+		)
+		(property "Value" "+3.3V"
+			(at 60.96 194.3099 90)
+			(effects
+				(font
+					(size 1.27 1.27)
+				)
+				(justify left)
+			)
+		)
+		(property "Footprint" ""
+			(at 64.77 194.31 0)
+			(effects
+				(font
+					(size 1.27 1.27)
+				)
+				(hide yes)
+			)
+		)
+		(property "Datasheet" ""
+			(at 64.77 194.31 0)
+			(effects
+				(font
+					(size 1.27 1.27)
+				)
+				(hide yes)
+			)
+		)
+		(property "Description" "Power symbol creates a global label with name \"+3.3V\""
+			(at 64.77 194.31 0)
+			(effects
+				(font
+					(size 1.27 1.27)
+				)
+				(hide yes)
+			)
+		)
+		(pin "1"
+		)
+		(instances
+			(project ""
+				(path "/9df24c09-b453-48f7-b96a-68d109fc3890"
+					(reference "#PWR040")
+					(unit 1)
+				)
